File: PCB/Kicad/CMT2119A.kicad_sch (KiCad schematic)
At the start: 11 parts, among them IC1 CMT2119A, J1 Conn_01x05_Pin, X1 NT3225SA 26 MHz

Commit message: Add files via upload
Parts:
- C3: value SOT -> 82pF
